File: BUS/KICAD/solar.cell.kicad_sch (KiCad schematic)
At the start: 3 parts

Commit message: Updated Bus
Parts:
- D5, D6: footprint (none) -> Diode_SMD:D_0603_1608Metric
- PV3: footprint (none) -> CUBESAT:SM811K08TF
Changed lines of the file:
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@@
 			)
 		)
-		(property "Footprint" ""
+		(property "Footprint" "CUBESAT:SM811K08TF"
 			(at 137.16 104.14 0)
 			(effects
@@
 			)
 		)
-		(property "Footprint" ""
+		(property "Footprint" "Diode_SMD:D_0603_1608Metric"
 			(at 170.18 104.14 0)
 			(effects
@@
 			)
 		)
-		(property "Footprint" ""
+		(property "Footprint" "Diode_SMD:D_0603_1608Metric"
 			(at 157.48 104.14 0)
 			(effects
