File: CONTROL/KICAD/magnetorquer.kicad_sch (KiCad schematic)
At the start: 2 parts, among them U4 DRV8210DRL

Commit message: Updated Control PCB / Schematics
Parts:
- removed L1: L, symbol Device:L
- removed U4: DRV8210DRL, symbol CUBESAT:DRV8210
- added C83: 100 nF, symbol Device:C
- added C84: ~, symbol Device:C
- added U22: DRV8212DRL, symbol CUBESAT:DRV8212
Connections:
- net V_GND: now also C83.2, C84.2, U22.3 (GND)
- new net IN_1: U22.1 (IN1)
- new net IN_2: U22.2 (IN2)
- new net OUT_1: U22.6 (OUT1)
- new net OUT_2: U22.4 (OUT2)
- new net V_BAT: C83.1, C84.1, U22.5 (VM)
Other:
- note added: "0 0 HI-Z HI-Z 1 1 L L 0 1 L H 1 0 H L"
- note added: "CURRENT CONTINOUS: 4 A PEAK: 8 A SLEEP: 84.5 nA"
- note added: "PWM: 0 ~ 100 kHz"
- note added: "VOLTAGE VM: 1.65 V ~ 11 V"
