File: CONTROL/KICAD/bldc_motor_driver.kicad_sch (KiCad schematic)
At the start: 12 parts, among them U6 MCT8316ZR

Commit message: Updated Control PCB / Schematics
Parts:
- removed C10: 22uF, symbol Device:C
- removed C11: 1uF, symbol Device:C
- removed C14: ~, symbol Device:C
- removed R3, R4, R5, R8: R, symbol Device:R
- added C21, C27, C28, C29: 100nF, symbol Device:C
- added C22: 22uF, symbol Device:C
- added C25: C_Polarized 10uF, symbol Device:C_Polarized
- added C26: 1uF, symbol Device:C
- added L2: 22uH, symbol Device:L
- added R13, R14, R15: 4.7kΩ, symbol Device:R
- C23: renamed from C12; value ~ -> 1uF
- U4: renamed from U6; footprint (none) -> Package_DFN_QFN:Texas_RGF_R-PVQFN-N40_EP3.7x5.7mm_ThermalVias
- renumbered C13 to C24, R6 to R16, R7 to R17
Connections:
- net V_3.3: now also R13.1, R14.1, R15.1
- net V_GND: now also C21.2, C22.2, C25.1, C26.2, C27.1, C28.1, C29.1
- net V_HV: now also C25.2, C27.2, C28.2, C29.2
- net V_AVDD: now reaches U4.25 (AVDD)
- net V_AVDD: now also C26.1
- net SPI.SDO: now reaches U4.33 (SDO)
- net SPI.SDO: now also R13.2
- net at R16.2, R17.1, U4.37 (ILIM): now also C21.1
- net CONTROL.FGOUT: now reaches U4.40 (FGOUT)
- net CONTROL.FGOUT: now also R15.2
- net CONTROL.FAULT: now reaches U4.22 (nFAULT)
- net CONTROL.FAULT: now also R14.2
- net at U4.3 (FB_BK): now also C22.1, L2.1
- net CONTROL.DRVOFF: now reaches U4.21 (DRVOFF)
- net CONTROL.SLEEP: now reaches U4.23 (nSLEEP)
- net SPI.SDI: now reaches U4.34 (SDI)
- net SPI.SCLK: now reaches U4.35 (SCLK)
- net SPI.CS: now reaches U4.36 (nSCS)
- net CONTROL.BRAKE: now reaches U4.38 (BRAKE)
- net CONTROL.PWM : now reaches U4.39 (PWM)
- net at U4.5 (SW_BK): now also L2.2
Other:
- note added: "AVDD: 10V"
- note added: "CAP VOLTAGE TWICE THE RATING"
- note added: "CP: 16V"
- note added: "HALL? BIPOLAR? UNIPOLAR? RATIOMETRIC?"
- note added: "PULL UP REQUIRED FOR SDO, FAULT, FGOUT"
- note added: "VERIFICATION SYMBOL: X SCHEMATIC: FOOTPRINT: BOARD:"
- note added: "VM: 24V"
- note removed: "BUCK COULD USE Inductor if we want"

Commit message: schematic design
Connections:
- net CONTROL.FAULT: no longer U4.22 (nFAULT)
- net CONTROL.FGOUT: no longer U4.40 (FGOUT)
- net CONTROL.BRAKE renamed BRAKE
- net CONTROL.DRVOFF renamed DRVOFF
- net CONTROL.PWM  renamed PWM
- net CONTROL.SLEEP renamed SLEEP
- new net FAULT: U4.22 (nFAULT)
- new net FGOUT: U4.40 (FGOUT)
Changed lines of the file:
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@@
 	(generator_version "8.0")
 	(paper "A4")
+	(bus_alias "PHASES"
+		(members "A" "B" "C")
+	)
 	(junction
 		(at 80.01 109.22)
@@
 	)
 	(bus_entry
-		(at 114.3 48.26)
+		(at 123.19 48.26)
 		(size 2.54 2.54)
 		(stroke
@@
 	)
 	(bus_entry
-		(at 114.3 60.96)
+		(at 123.19 60.96)
 		(size 2.54 2.54)
 		(stroke
@@
 	)
 	(bus_entry
-		(at 114.3 68.58)
+		(at 123.19 68.58)
 		(size 2.54 2.54)
 		(stroke
@@
 	)
 	(bus_entry
-		(at 114.3 50.8)
+		(at 123.19 50.8)
 		(size 2.54 2.54)
 		(stroke
@@
 	)
 	(bus_entry
-		(at 114.3 71.12)
+		(at 123.19 71.12)
 		(size 2.54 2.54)
 		(stroke
@@
 	)
 	(bus_entry
-		(at 114.3 58.42)
+		(at 123.19 58.42)
 		(size 2.54 2.54)
 		(stroke
@@
 	(wire
 		(pts
-			(xy 116.84 63.5) (xy 137.16 63.5)
+			(xy 125.73 63.5) (xy 137.16 63.5)
 		)
 		(stroke
@@
 	(wire
 		(pts
-			(xy 116.84 60.96) (xy 137.16 60.96)
+			(xy 125.73 60.96) (xy 137.16 60.96)
 		)
 		(stroke
@@
 	(bus
 		(pts
-			(xy 59.69 41.91) (xy 114.3 41.91)
+			(xy 107.95 41.91) (xy 123.19 41.91)
 		)
 		(stroke
@@
 	(bus
 		(pts
-			(xy 181.61 96.52) (xy 198.12 96.52)
+			(xy 181.61 96.52) (xy 199.39 96.52)
 		)
 		(stroke
@@
 	(bus
 		(pts
-			(xy 114.3 60.96) (xy 114.3 68.58)
+			(xy 123.19 60.96) (xy 123.19 68.58)
 		)
 		(stroke
@@
 	(wire
 		(pts
-			(xy 116.84 50.8) (xy 137.16 50.8)
+			(xy 125.73 50.8) (xy 137.16 50.8)
 		)
 		(stroke
@@
 	(wire
 		(pts
-			(xy 116.84 71.12) (xy 137.16 71.12)
+			(xy 125.73 71.12) (xy 137.16 71.12)
 		)
 		(stroke
@@
 	(wire
 		(pts
-			(xy 116.84 73.66) (xy 137.16 73.66)
+			(xy 125.73 73.66) (xy 137.16 73.66)
 		)
 		(stroke
@@
 	(bus
 		(pts
-			(xy 93.98 76.2) (xy 120.65 76.2)
+			(xy 111.76 76.2) (xy 120.65 76.2)
 		)
 		(stroke
@@
 	(bus
 		(pts
-			(xy 114.3 41.91) (xy 114.3 48.26)
+			(xy 123.19 41.91) (xy 123.19 48.26)
 		)
 		(stroke
@@
 	(bus
 		(pts
-			(xy 114.3 68.58) (xy 114.3 71.12)
+			(xy 123.19 68.58) (xy 123.19 71.12)
 		)
 		(stroke
@@
 	(bus
 		(pts
-			(xy 114.3 48.26) (xy 114.3 50.8)
+			(xy 123.19 48.26) (xy 123.19 50.8)
 		)
 		(stroke
@@
 	(bus
 		(pts
-			(xy 114.3 50.8) (xy 114.3 58.42)
+			(xy 123.19 50.8) (xy 123.19 58.42)
 		)
 		(stroke
@@
 	(bus
 		(pts
-			(xy 185.42 45.72) (xy 204.47 45.72)
+			(xy 185.42 45.72) (xy 205.74 45.72)
 		)
 		(stroke
@@
 	(bus
 		(pts
-			(xy 114.3 58.42) (xy 114.3 60.96)
+			(xy 123.19 58.42) (xy 123.19 60.96)
 		)
 		(stroke
@@
 	(wire
 		(pts
-			(xy 116.84 53.34) (xy 137.16 53.34)
+			(xy 125.73 53.34) (xy 137.16 53.34)
 		)
 		(stroke
@@
 		)
 	)
-	(label "CONTROL.BRAKE"
+	(label "BRAKE"
 		(at 134.62 73.66 180)
 		(fields_autoplaced yes)
@@
 		)
 	)
-	(label "CONTROL.DRVOFF"
+	(label "DRVOFF"
 		(at 134.62 60.96 180)
 		(fields_autoplaced yes)
@@
 		)
 	)
-	(label "CONTROL{BRAKE PWM FAULT SLEEP DRVOFF FGOUT}"
-		(at 62.23 41.91 0)
-		(fields_autoplaced yes)
-		(effects
-			(font
-				(size 1.27 1.27)
-			)
-			(justify left bottom)
+	(label "{CONTROL}"
+		(at 120.65 41.91 180)
+		(fields_autoplaced yes)
+		(effects
+			(font
+				(size 1.27 1.27)
+			)
+			(justify right bottom)
 		)
 	)
@@
 		)
 	)
-	(label "CONTROL.SLEEP"
+	(label "SLEEP"
 		(at 134.62 53.34 180)
 		(fields_autoplaced yes)
@@
 		)
 	)
-	(label "CONTROL.FAULT"
+	(label "FAULT"
 		(at 134.62 50.8 180)
 		(fields_autoplaced yes)
@@
 		)
 	)
-	(label "SPI{CS SCLK SDI SDO}"
+	(label "{SPI}"
 		(at 118.11 76.2 180)
 		(fields_autoplaced yes)
@@
 		)
 	)
-	(label "CONTROL.FGOUT"
+	(label "FGOUT"
 		(at 134.62 63.5 180)
 		(fields_autoplaced yes)
@@
 		)
 	)
-	(label "MOTOR{A B C}"
+	(label "MOTOR{PHASES}"
 		(at 187.96 45.72 0)
 		(fields_autoplaced yes)
@@
 		)
 	)
-	(label "HALL{A B C}"
+	(label "HALL{PHASES}"
 		(at 184.15 96.52 0)
 		(fields_autoplaced yes)
@@
 		)
 	)
-	(label "CONTROL.PWM "
+	(label "PWM"
 		(at 134.62 71.12 180)
 		(fields_autoplaced yes)
@@
 		)
 	)
-	(hierarchical_label "HALL{A  B C} "
-		(shape input)
-		(at 198.12 96.52 0)
+	(hierarchical_label "HALL{PHASES} "
+		(shape input)
+		(at 199.39 96.52 0)
 		(fields_autoplaced yes)
 		(effects
@@
 		)
 	)
-	(hierarchical_label "MOTOR{A B C}"
+	(hierarchical_label "MOTOR{PHASES}"
 		(shape output)
-		(at 204.47 45.72 0)
+		(at 205.74 45.72 0)
 		(fields_autoplaced yes)
 		(effects
@@
 		)
 	)
-	(hierarchical_label "CONTROL{BRAKE PWM FAULT SLEEP DRVOFF FGOUT}"
+	(hierarchical_label "{CONTROL}"
 		(shape bidirectional)
-		(at 59.69 41.91 180)
+		(at 107.95 41.91 180)
 		(fields_autoplaced yes)
 		(effects
@@
 		)
 	)
-	(hierarchical_label "SPI{CS SCLK SDI SDO}"
+	(hierarchical_label "{SPI}"
 		(shape bidirectional)
-		(at 93.98 76.2 180)
-		(fields_autoplaced yes)
-		(effects
+		(at 111.76 76.2 180)
+		(fields_autoplaced yes)
+		(effects
