File: CONTROL/KICAD/imu.kicad_sch (KiCad schematic)
At the start: 3 parts

Commit message: Updated Control PCB / Schematics
Parts:
- removed U2: ~, symbol CUBESAT:LSM6DSO
- added R26, R27: 0Ω, symbol Device:R
- added U9: LSM6DSO, symbol CUBESAT:LSM6DSO
- renumbered C4 to C38, C5 to C39
Connections:
- net INT1: now also U9.4 (INT1)
- net INT2: now also U9.9 (INT2)
- net V_GND: now also R27.2, U9.2 (SDX), U9.3 (SCX), U9.6 (GND), U9.7 (GND)
- net V_LV renamed V_3.3
- net V_3.3: now also R26.1, U9.12 (CS), U9.5 (VDD_IO), U9.8 (VDD)
- new net: R26.2, R27.1, U9.1 (SDO/SA0)
- new net ISC.SCL: U9.13 (SCL/SPC)
- new net ISC.SDA: U9.14 (SDA/SDI/SDO)
Other:
- note added: "ADDRESS 0: 6A 1: 6B"
- note added: "CS HIGH = I2C"
- note added: "VERIFICATION SYMBOL: X SCHEMATIC: X FOOTPRINT: BOARD:"
- moved on the sheet: C38, C39

Commit message: schematic design
Parts:
- renumbered C38 to C70, C39 to C71, R26 to R77, R27 to R78, U9 to U16
Connections:
- net ISC.SCL renamed SCL
- net ISC.SDA renamed SDA
Changed lines of the file:
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@@
 	)
 	(bus_entry
-		(at 105.41 81.28)
+		(at 113.03 81.28)
 		(size 2.54 2.54)
 		(stroke
@@
 	)
 	(bus_entry
-		(at 105.41 83.82)
+		(at 113.03 83.82)
 		(size 2.54 2.54)
 		(stroke
@@
 	(wire
 		(pts
-			(xy 107.95 83.82) (xy 124.46 83.82)
-		)
-		(stroke
-			(width 0)
-			(type default)
-		)
-	)
-	(wire
-		(pts
 			(xy 152.4 104.14) (xy 152.4 101.6)
 		)
@@
 	(wire
 		(pts
+			(xy 115.57 83.82) (xy 124.46 83.82)
+		)
+		(stroke
+			(width 0)
+			(type default)
+		)
+	)
+	(wire
+		(pts
 			(xy 121.92 101.6) (xy 124.46 101.6)
 		)
@@
 	(bus
 		(pts
-			(xy 105.41 60.96) (xy 105.41 81.28)
+			(xy 113.03 81.28) (xy 113.03 83.82)
 		)
 		(stroke
@@
 	(bus
 		(pts
-			(xy 90.17 60.96) (xy 105.41 60.96)
+			(xy 110.49 78.74) (xy 113.03 78.74)
 		)
 		(stroke
@@
 	(bus
 		(pts
-			(xy 105.41 81.28) (xy 105.41 83.82)
+			(xy 113.03 78.74) (xy 113.03 81.28)
 		)
 		(stroke
@@
 	(wire
 		(pts
-			(xy 107.95 86.36) (xy 124.46 86.36)
+			(xy 115.57 86.36) (xy 124.46 86.36)
 		)
 		(stroke
@@
 		)
 	)
-	(label "ISC{SDA SCL}"
-		(at 105.41 60.96 180)
+	(label "SCL"
+		(at 121.92 83.82 180)
 		(fields_autoplaced yes)
 		(effects
@@
 		)
 	)
-	(label "ISC.SCL"
-		(at 121.92 83.82 180)
+	(label "SDA"
+		(at 121.92 86.36 180)
 		(fields_autoplaced yes)
 		(effects
@@
 		)
 	)
-	(label "ISC.SDA"
-		(at 121.92 86.36 180)
-		(fields_autoplaced yes)
-		(effects
-			(font
-				(size 1.27 1.27)
-			)
-			(justify right bottom)
-		)
-	)
 	(hierarchical_label "V_3.3"
 		(shape input)
@@
 		)
 	)
-	(hierarchical_label "I2C"
+	(hierarchical_label "{I2C}"
 		(shape bidirectional)
-		(at 90.17 60.96 180)
+		(at 110.49 78.74 180)
 		(fields_autoplaced yes)
 		(effects
@@
 		(dnp no)
 		(fields_autoplaced yes)
-		(property "Reference" "R27"
+		(property "Reference" "R78"
 			(at 100.33 93.9799 0)
 			(effects
@@
 		(dnp yes)
 		(fields_autoplaced yes)
-		(property "Reference" "R26"
+		(property "Reference" "R77"
 			(at 100.33 81.2799 0)
 			(effects
@@
 		(dnp no)
 		(fields_autoplaced yes)
-		(property "Reference" "C38"
+		(property "Reference" "C70"
 			(at 54.61 99.0599 0)
 			(effects
@@
 		(dnp no)
 		(fields_autoplaced yes)
-		(property "Reference" "C39"
+		(property "Reference" "C71"
 			(at 67.31 99.0599 0)
 			(effects
@@
 		(dnp no)
 		(fields_autoplaced yes)
-		(property "Reference" "U9"
+		(property "Reference" "U16"
 			(at 137.16 75.946 0)
 			(do_not_autoplace yes)
