File: CONTROL/KICAD/magnetometer.kicad_sch (KiCad schematic)
At the start: 4 parts

Commit message: Updated Control PCB / Schematics
Parts:
- removed C8: 100nF, symbol Device:C
- removed U3: ~, symbol CUBESAT:LIS3DML
- added C37: 100nF, symbol Device:C
- added R24, R25: 0Ω, symbol Device:R
- added U8: LIS3MDL, Package_LGA:LGA-12_2x2mm_P0.5mm, symbol CUBESAT:LIS3DML
- renumbered C6 to C35, C7 to C36
Connections:
- net V_GND: now also C37.2, R25.2, U8.12 (RESERVED), U8.2 (RESERVED), U8.3 (GND)
- net V_LV renamed V_3.3
- net V_3.3: now also R24.1, U8.10 (CS), U8.5 (VDD), U8.6 (VDD_IO)
- new net: C37.1, U8.4 (C1)
- new net: R24.2, R25.1, U8.9 (SDO/SA1)
- new net DRDY: U8.8 (DRDY)
- new net I2C.SCL: U8.1 (SCL/SPL)
- new net I2C.SDA: U8.11 (SDA/SDI/SDO)
- new net INT: U8.7 (INT)
Other:
- note added: "ADDRESS 0: 1C 1: 1E"
- note added: "CS HIGH = I2C"
- note added: "VERIFICATION SYMBOL: X SCHEMATIC: X FOOTPRINT: BOARD:"
- moved on the sheet: C35, C36

Commit message: schematic design
Parts:
- renumbered C35 to C72, C36 to C73, C37 to C74, R24 to R79, R25 to R80, U8 to U17
Connections:
- net I2C.SCL renamed SCL
- net I2C.SDA renamed SDA
Changed lines of the file:
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@@
 	)
 	(bus_entry
-		(at 92.71 96.52)
+		(at 100.33 96.52)
 		(size 2.54 2.54)
 		(stroke
@@
 	)
 	(bus_entry
-		(at 92.71 99.06)
+		(at 100.33 99.06)
 		(size 2.54 2.54)
 		(stroke
@@
 	(bus
 		(pts
-			(xy 74.93 76.2) (xy 92.71 76.2)
+			(xy 97.79 93.98) (xy 100.33 93.98)
 		)
 		(stroke
@@
 	(wire
 		(pts
-			(xy 95.25 99.06) (xy 111.76 99.06)
+			(xy 102.87 99.06) (xy 111.76 99.06)
 		)
 		(stroke
@@
 	(bus
 		(pts
-			(xy 92.71 76.2) (xy 92.71 96.52)
+			(xy 100.33 93.98) (xy 100.33 96.52)
 		)
 		(stroke
@@
 	(bus
 		(pts
-			(xy 92.71 96.52) (xy 92.71 99.06)
+			(xy 100.33 96.52) (xy 100.33 99.06)
 		)
 		(stroke
@@
 	(wire
 		(pts
-			(xy 95.25 101.6) (xy 111.76 101.6)
+			(xy 102.87 101.6) (xy 111.76 101.6)
 		)
 		(stroke
@@
 		)
 	)
-	(label "I2C{SDA SCL}"
-		(at 90.17 76.2 180)
+	(label "SDA"
+		(at 109.22 101.6 180)
 		(fields_autoplaced yes)
 		(effects
@@
 		)
 	)
-	(label "I2C.SDA"
-		(at 109.22 101.6 180)
-		(fields_autoplaced yes)
-		(effects
-			(font
-				(size 1.27 1.27)
-			)
-			(justify right bottom)
-		)
-	)
-	(label "I2C.SCL"
+	(label "SCL"
 		(at 109.22 99.06 180)
 		(fields_autoplaced yes)
@@
 		)
 	)
-	(hierarchical_label "I2C"
+	(hierarchical_label "{I2C}"
 		(shape bidirectional)
-		(at 74.93 76.2 180)
+		(at 97.79 93.98 180)
 		(fields_autoplaced yes)
 		(effects
@@
 		(dnp no)
 		(fields_autoplaced yes)
-		(property "Reference" "C36"
+		(property "Reference" "C73"
 			(at 71.12 101.5999 0)
 			(effects
@@
 		(on_board yes)
 		(dnp no)
-		(property "Reference" "C37"
+		(property "Reference" "C74"
 			(at 158.75 119.3801 0)
 			(effects
@@
 		(dnp no)
 		(fields_autoplaced yes)
-		(property "Reference" "C35"
+		(property "Reference" "C72"
 			(at 58.42 101.5999 0)
 			(effects
@@
 		(dnp yes)
 		(fields_autoplaced yes)
-		(property "Reference" "R24"
+		(property "Reference" "R79"
 			(at 86.36 96.5199 0)
 			(effects
@@
 		(on_board yes)
 		(dnp no)
-		(property "Reference" "U8"
+		(property "Reference" "U17"
 			(at 125.73 91.186 0)
 			(do_not_autoplace yes)
@@
 		(dnp no)
 		(fields_autoplaced yes)
-		(property "Reference" "R25"
+		(property "Reference" "R80"
 			(at 86.36 109.2199 0)
 			(effects
