File: CONTROL/KICAD/magnetorquers.kicad_sch (KiCad schematic)
At the start: 0 parts

Commit message: schematic design
Connections:
- no-connect marks 4 -> 0
Other:
- added sheet EFUSE_LATCHED1 (../../POWER/KICAD/efuse.latched.kicad_sch)
- added sheet EFUSE_LATCHED2 (../../POWER/KICAD/efuse.latched.kicad_sch)
- added sheet EFUSE_LATCHED3 (../../POWER/KICAD/efuse.latched.kicad_sch)
- sheet COMMAND1 ports: added V_IN, {CAN}, {I2C}, {PA}, {PB}, {PC}, {PD}, {PE}, {PH}; removed CAN{H L}, I2C{SCL SDA}, PA[0..15], PB[0..15], PC[0..15], PD[0..15], PE[0..15], PH[0..3], V_LV
- sheet IMU 2 ports: added {I2C}; removed I2C
- sheet MAGNETOMETER 2 ports: added {I2C}; removed I2C
- note added: "INCLUDED ARE TEST POINTS / PADS TO SOLDER IN CASE THE MAGNETORQUERS ARE TOO WEAK"
