File: CONTROL/KICAD/reaction_wheel.kicad_sch (KiCad schematic)
At the start: 4 parts

Commit message: schematic design
Parts:
- removed R28, R29, R30: 0Ω, Resistor_SMD:R_0603_1608Metric, symbol Device:R
Connections:
- net MONITOR1/IN renamed EFUSE_LATCHED/V_OUT
Other:
- added sheet EFUSE_LATCHED (../../POWER/KICAD/efuse.latched.kicad_sch)
- sheet BLDC_MOTOR_DRIVER ports: added HALL{PHASES}, MOTOR{PHASES}, {CONTROL}, {SPI}; removed CONTROL, HALL, MOTOR, SPI
- sheet MONITOR1 ports: added {I2C}; removed I2C
