File: CONTROL/KICAD/reaction_wheels.kicad_sch (KiCad schematic)
At the start: 2 parts

Commit message: schematic design
Other:
- sheet COMMAND ports: added {CAN}, {I2C}, {PA}, {PB}, {PC}, {PD}, {PE}, {PH}; removed CAN{H L}, I2C{SCL SDA}, PA[0..15], PB[0..15], PC[0..15], PD[0..15], PE[0..15], PH[0..3]
- sheet IMU 1 ports: added {I2C}; removed I2C
- sheet MAGNETOMETER 1 ports: added {I2c}; removed I2C
- sheet REACTION WHEEL 3 ports: added CONTROL_4{CONTROL}, {SPI}; removed CONTROL, SPI
- sheet REACTION WHEEL 4 ports: added {SPI}; removed SPI
Changed lines of the file:
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@@
-		)
-	)
-	(label "PE[0..15]"
-		(at 83.82 96.52 0)
-		(fields_autoplaced yes)
-		(effects
-			(font
-				(size 1.27 1.27)
-			)
-			(justify left bottom)
 		)
 	)
@@
 		)
 	)
-	(label "PA[0..15]"
-		(at 83.82 86.36 0)
-		(fields_autoplaced yes)
-		(effects
-			(font
-				(size 1.27 1.27)
-			)
-			(justify left bottom)
-		)
-	)
 	(label "CONTROL_2{BRAKE PWM FAULT SLEEP DRVOFF FGOUT}"
 		(at 163.83 62.23 180)
@@
 		)
 	)
-	(label "CONTROL_4{BRAKE PWM FAULT SLEEP DRVOFF FGOUT}"
-		(at 198.12 133.35 180)
-		(fields_autoplaced yes)
-		(effects
-			(font
-				(size 1.27 1.27)
-			)
-			(justify right bottom)
-		)
-	)
 	(label "I2C3"
 		(at 78.74 151.13 180)
@@
 		)
 	)
-	(label "PD[0..15]"
-		(at 83.82 93.98 0)
-		(fields_autoplaced yes)
-		(effects
-			(font
-				(size 1.27 1.27)
-			)
-			(justify left bottom)
-		)
-	)
 	(label "I2C3"
 		(at 163.83 120.65 180)
@@
 		)
 	)
-	(label "PC[0..15]"
-		(at 83.82 91.44 0)
-		(fields_autoplaced yes)
-		(effects
-			(font
-				(size 1.27 1.27)
-			)
-			(justify left bottom)
-		)
-	)
-	(label "PB[0..15]"
-		(at 83.82 88.9 0)
-		(fields_autoplaced yes)
-		(effects
-			(font
-				(size 1.27 1.27)
-			)
-			(justify left bottom)
-		)
-	)
 	(label "I2C3"
 		(at 78.74 170.18 180)
@@
 		)
 	)
-	(label "PH[0..3]"
-		(at 83.82 99.06 0)
-		(fields_autoplaced yes)
-		(effects
-			(font
-				(size 1.27 1.27)
-			)
-			(justify left bottom)
-		)
-	)
 	(label "I2C3"
 		(at 163.83 67.31 180)
@@
 		)
 	)
-	(hierarchical_label "CAN{H L}"
+	(hierarchical_label "{CAN}"
 		(shape bidirectional)
 		(at 34.29 87.63 180)
@@
 		)
 	)
-	(hierarchical_label "I2C{SCL SDA}"
+	(hierarchical_label "{I2C}"
 		(shape bidirectional)
 		(at 34.29 90.17 180)
@@
 			)
 		)
-		(pin "SPI" bidirectional
+		(pin "{SPI}" bidirectional
 			(at 166.37 118.11 180)
 			(effects
@@
 			)
 		)
-		(pin "I2C{SCL SDA}" bidirectional
+		(pin "{I2C}" bidirectional
 			(at 36.83 90.17 180)
 			(effects
@@
 			)
 		)
-		(pin "CAN{H L}" input
+		(pin "{CAN}" input
 			(at 36.83 87.63 180)
 			(effects
@@
 				)
 				(justify left)
-			)
-		)
-		(pin "PD[0..15]" bidirectional
-			(at 81.28 93.98 0)
-			(effects
-				(font
-					(size 1.27 1.27)
-				)
-				(justify right)
-			)
-		)
-		(pin "PB[0..15]" bidirectional
-			(at 81.28 88.9 0)
-			(effects
-				(font
-					(size 1.27 1.27)
-				)
-				(justify right)
-			)
-		)
-		(pin "PH[0..3]" bidirectional
-			(at 81.28 99.06 0)
-			(effects
-				(font
-					(size 1.27 1.27)
-				)
-				(justify right)
-			)
-		)
-		(pin "PC[0..15]" bidirectional
-			(at 81.28 91.44 0)
-			(effects
-				(font
-					(size 1.27 1.27)
-				)
-				(justify right)
-			)
-		)
-		(pin "PA[0..15]" bidirectional
-			(at 81.28 86.36 0)
-			(effects
-				(font
-					(size 1.27 1.27)
-				)
-				(justify right)
 			)
 		)
@@
 			)
 		)
-		(pin "PE[0..15]" bidirectional
+		(pin "{PD}" bidirectional
+			(at 81.28 93.98 0)
+			(effects
+				(font
+					(size 1.27 1.27)
+				)
+				(justify right)
+			)
+		)
+		(pin "{PB}" bidirectional
+			(at 81.28 88.9 0)
+			(effects
+				(font
+					(size 1.27 1.27)
+				)
+				(justify right)
+			)
+		)
+		(pin "{PA}" bidirectional
+			(at 81.28 86.36 0)
+			(effects
+				(font
+					(size 1.27 1.27)
+				)
+				(justify right)
+			)
+		)
+		(pin "{PC}" bidirectional
+			(at 81.28 91.44 0)
+			(effects
+				(font
+					(size 1.27 1.27)
+				)
+				(justify right)
+			)
+		)
+		(pin "{PE}" bidirectional
 			(at 81.28 96.52 0)
+			(effects
+				(font
+					(size 1.27 1.27)
+				)
+				(justify right)
+			)
+		)
+		(pin "{PH}" bidirectional
+			(at 81.28 99.06 0)
 			(effects
 				(font
@@
 			)
 		)
-		(pin "I2C" bidirectional
+		(pin "{I2c}" bidirectional
 			(at 81.28 170.18 180)
 			(effects
@@
 			)
 		)
-		(pin "I2C" bidirectional
+		(pin "{I2C}" bidirectional
 			(at 81.28 151.13 180)
 			(effects
@@
 			)
 		)
-		(pin "SPI" bidirectional
+		(pin "{SPI}" bidirectional
 			(at 166.37 91.44 180)
 			(effects
@@
 			)
 		)
-		(pin "CONTROL" bidirectional
+		(pin "CONTROL_4{CONTROL}" bidirectional
 			(at 166.37 88.9 180)
 			(effects
