File: COMMAND/KICAD/can.kicad_sch (KiCad schematic)
At the start: 3 parts

Commit message: Updated Command Kicad
Parts:
- removed U?: TCANC3403-Q1, symbol CUBESAT:TCANC3403-Q1
- added U6: TCAN3403-Q1, Package_DFN_QFN:Texas_DRB0008J, symbol CUBESAT:TCANC3403DR-Q1
- C31, C32: renamed from C?; footprint (none) -> Capacitor_SMD:C_0603_1608Metric
Connections:
- net CAN.H: now also U6.7 (CAN_H)
- net CAN.L: now also U6.6 (CAN_L)
- net V_GND: now also U6.2 (GND)
- net V_LV renamed V_3.3
- net V_3.3: now also U6.3 (VCC), U6.5 (V_IO)
- new net CAN_I.RX: U6.4 (RXD)
- new net CAN_I.TX: U6.1 (TXD)
- new net STB: U6.8 (STB)
Other:
- note added: "DECOUPLING CAPS"
- note added: "VERIFICATION SYMBOL: X SCHEMATIC: X FOOTPRINT: X BOARD:"
- moved on the sheet: C31, C32

Commit message: schematic design
Parts:
- removed U6: TCAN3403-Q1, Package_DFN_QFN:Texas_DRB0008J, symbol CUBESAT:TCANC3403DR-Q1
- added U5: TCAN3413DDFR, Package_DFN_QFN:Texas_DRB0008J, symbol CUBESAT:TCANC3413DDF
Connections:
- net CAN_I.RX: now also U5.4 (RXD)
- net CAN_I.TX: now also U5.1 (TXD)
- net STB: now also U5.8 (STB)
- net V_3.3: now also U5.3 (VCC), U5.5 (V_IO)
- net V_GND: now also U5.2 (GND)
- new net H: U5.7 (CAN_H)
- new net L: U5.6 (CAN_L)
Other:
- note added: "CAN UNPOWERED: HI-Z"
- note added: "STANDBY PULL UP ACTIVE HIGH"
- note removed: "CAN IS HI-Z WHEN UNPOWERED"
- note removed: "STANDBY IS ACTIVE HIGH"
- note removed: "STB HAS PULLUP"
Changed lines of the file:
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@@
 	)
 	(bus_entry
-		(at 179.07 95.25)
+		(at 175.26 95.25)
 		(size -2.54 2.54)
 		(stroke
@@
 	)
 	(bus_entry
-		(at 179.07 97.79)
+		(at 175.26 97.79)
 		(size -2.54 2.54)
 		(stroke
@@
 	(wire
 		(pts
-			(xy 166.37 100.33) (xy 176.53 100.33)
+			(xy 166.37 100.33) (xy 172.72 100.33)
+		)
+		(stroke
+			(width 0)
+			(type default)
+		)
+	)
+	(bus
+		(pts
+			(xy 175.26 91.44) (xy 185.42 91.44)
 		)
 		(stroke
@@
 	(bus
 		(pts
-			(xy 179.07 95.25) (xy 179.07 97.79)
+			(xy 175.26 95.25) (xy 175.26 97.79)
 		)
 		(stroke
@@
 		)
 	)
+	(wire
+		(pts
+			(xy 166.37 97.79) (xy 172.72 97.79)
+		)
+		(stroke
+			(width 0)
+			(type default)
+		)
+	)
+	(wire
+		(pts
+			(xy 144.78 105.41) (xy 147.32 105.41)
+		)
+		(stroke
+			(width 0)
+			(type default)
+		)
+	)
 	(bus
 		(pts
-			(xy 191.77 91.44) (xy 179.07 91.44)
-		)
-		(stroke
-			(width 0)
-			(type default)
-		)
-	)
-	(wire
-		(pts
-			(xy 166.37 97.79) (xy 176.53 97.79)
-		)
-		(stroke
-			(width 0)
-			(type default)
-		)
-	)
-	(wire
-		(pts
-			(xy 144.78 105.41) (xy 147.32 105.41)
+			(xy 133.35 95.25) (xy 133.35 92.71)
 		)
 		(stroke
@@
 	(bus
 		(pts
-			(xy 133.35 95.25) (xy 133.35 92.71)
+			(xy 175.26 91.44) (xy 175.26 95.25)
+		)
+		(stroke
+			(width 0)
+			(type default)
+		)
+	)
+	(wire
+		(pts
+			(xy 144.78 110.49) (xy 147.32 110.49)
+		)
+		(stroke
+			(width 0)
+			(type default)
+		)
+	)
+	(wire
+		(pts
+			(xy 78.74 99.06) (xy 78.74 96.52)
+		)
+		(stroke
+			(width 0)
+			(type default)
+		)
+	)
+	(wire
+		(pts
+			(xy 78.74 109.22) (xy 78.74 106.68)
+		)
+		(stroke
+			(width 0)
+			(type default)
+		)
+	)
+	(wire
+		(pts
+			(xy 144.78 113.03) (xy 147.32 113.03)
 		)
 		(stroke
@@
 	(bus
 		(pts
-			(xy 179.07 91.44) (xy 179.07 95.25)
-		)
-		(stroke
-			(width 0)
-			(type default)
-		)
-	)
-	(wire
-		(pts
-			(xy 144.78 110.49) (xy 147.32 110.49)
-		)
-		(stroke
-			(width 0)
-			(type default)
-		)
-	)
-	(wire
-		(pts
-			(xy 78.74 99.06) (xy 78.74 96.52)
-		)
-		(stroke
-			(width 0)
-			(type default)
-		)
-	)
-	(wire
-		(pts
-			(xy 78.74 109.22) (xy 78.74 106.68)
-		)
-		(stroke
-			(width 0)
-			(type default)
-		)
-	)
-	(wire
-		(pts
-			(xy 144.78 113.03) (xy 147.32 113.03)
-		)
-		(stroke
-			(width 0)
-			(type default)
-		)
-	)
-	(bus
-		(pts
 			(xy 115.57 92.71) (xy 133.35 92.71)
 		)
@@
 	)
 	(rectangle
-		(start 58.42 83.82)
-		(end 100.33 121.92)
+		(start 59.055 83.185)
+		(end 100.965 121.285)
 		(stroke
 			(width 0)
@@
 		)
 	)
-	(text "STB HAS PULLUP"
+	(text "STANDBY\n	PULL UP\n	ACTIVE HIGH"
 		(exclude_from_sim no)
-		(at 114.3 86.36 0)
+		(at 119.38 63.5 0)
 		(effects
 			(font
@@
 		)
 	)
-	(text "CAN IS HI-Z WHEN UNPOWERED\n"
+	(text "CAN\n	UNPOWERED: HI-Z"
 		(exclude_from_sim no)
-		(at 170.18 86.36 0)
+		(at 172.72 78.74 0)
 		(effects
 			(font
@@
 	(text "DECOUPLING CAPS"
 		(exclude_from_sim no)
-		(at 62.23 86.36 0)
+		(at 60.96 86.36 0)
 		(effects
 			(font
@@
 		)
 	)
-	(text "VERIFICATION\nSYMBOL: X\nSCHEMATIC: X\nFOOTPRINT: X\nBOARD: "
+	(text "VERIFICATION\n	SYMBOL: X\n	SCHEMATIC: X\n	FOOTPRINT: X\n	BOARD: "
 		(exclude_from_sim no)
-		(at 163.83 64.008 0)
+		(at 119.38 71.12 0)
 		(effects
 			(font
@@
 			)
 			(justify left top)
-		)
-	)
-	(text "STANDBY IS ACTIVE HIGH"
-		(exclude_from_sim no)
-		(at 114.3 84.328 0)
-		(effects
-			(font
-				(size 1.27 1.27)
-			)
-			(justify left)
 		)
 	)
@@
 		)
 	)
-	(label "CAN_O{H L}"
-		(at 179.07 91.44 0)
+	(label "{CAN}"
+		(at 177.8 91.44 0)
 		(fields_autoplaced yes)
 		(effects
@@
 		)
 	)
-	(label "CAN.H"
+	(label "H"
 		(at 168.91 97.79 0)
 		(fields_autoplaced yes)
@@
 		)
 	)
-	(label "CAN.L"
+	(label "L"
 		(at 168.91 100.33 0)
 		(fields_autoplaced yes)
@@
 		)
 	)
-	(hierarchical_label "CAN_O{H L}"
-		(shape input)
-		(at 191.77 91.44 0)
+	(hierarchical_label "{CAN}"
+		(shape input)
+		(at 185.42 91.44 0)
 		(fields_autoplaced yes)
 		(effects
@@
 	)
 	(symbol
-		(lib_id "CUBESAT:TCANC3403DR-Q1")
+		(lib_id "CUBESAT:TCANC3413DDF")
 		(at 156.21 105.41 0)
 		(unit 1)
@@
 		(dnp no)
 		(fields_autoplaced yes)
-		(property "Reference" "U6"
+		(property "Reference" "U5"
 			(at 156.845 90.17 0)
 			(effects
@@
 			)
 		)
-		(property "Value" "TCAN3403-Q1"
+		(property "Value" "TCAN3413DDFR"
 			(at 156.845 92.71 0)
 			(effects
@@
 		)
 		(property "Footprint" "Package_DFN_QFN:Texas_DRB0008J"
-			(at 147.32 97.79 0)
-			(effects
-				(font
-					(size 1.27 1.27)
-				)
-				(hide yes)
-			)
-		)
-		(property "Datasheet" "https://www.ti.com/lit/ds/symlink/tcan3403-q1.pdf"
-			(at 190.5 95.25 0)
-			(effects
-				(font
-					(size 1.27 1.27)
-				)
-				(hide yes)
-			)
-		)
-		(property "Description" "TCAN340x-Q1 3.3V Automotive CAN FD Transceivers with Standby Mode and ±58V bus Standoff"
+			(at 156.464 105.156 0)
+			(effects
+				(font
+					(size 1.27 1.27)
+				)
+				(hide yes)
+			)
+		)
+		(property "Datasheet" "https://www.ti.com/lit/ds/symlink/tcan3413.pdf"
+			(at 156.21 105.41 0)
+			(effects
+				(font
+					(size 1.27 1.27)
+				)
+				(hide yes)
+			)
+		)
+		(property "Description" "TCAN340x 3.3V CAN FD Transceivers with Standby Mode and ±58V bus Standoff"
 			(at 203.708 75.692 0)
 			(effects
@@
 			)
 		)
+		(pin "7"
+		)
+		(pin "5"
+		)
+		(pin "8"
+		)
+		(pin "2"
+		)
 		(pin "1"
 		)
-		(pin "2"
+		(pin "6"
+		)
+		(pin "4"
 		)
 		(pin "3"
-		)
-		(pin "4"
-		)
-		(pin "6"
-		)
-		(pin "5"
-		)
-		(pin "8"
-		)
-		(pin "7"
 		)
 		(instances
 			(project "control"
-				(path "/c4b3c8f9-82bd-4648-8d22-870bf16aa829/29a81977-0a76-472b-8d88-45695e75b501/ace0dddc-e7de-4238-9577-ce744b7cdb3f/3f2d8199-33e9-456c-b5a1-16126a4e29ed"
-					(reference "U21")
-					(unit 1)
-				)
-				(path "/c4b3c8f9-82bd-4648-8d22-870bf16aa829/94383bfe-d869-4ac9-b660-9c199e344f31/9d3a0f9f-9dfc-4311-9915-9308a3fac81f/3f2d8199-33e9-456c-b5a1-16126a4e29ed"
-					(reference "U6")
+				(path "/c4b3c8f9-82bd-4648-8d22-870bf16aa829/29a81977-0a76-472b-8d88-45695e75b501/5d95f24e-69a0-4585-974a-64f0c2602c3c/fd3f1189-33c7-4694-b893-b6769cf32056"
+					(reference "U5")
+					(unit 1)
+				)
+				(path "/c4b3c8f9-82bd-4648-8d22-870bf16aa829/94383bfe-d869-4ac9-b660-9c199e344f31/9d3a0f9f-9dfc-4311-9915-9308a3fac81f/fd3f1189-33c7-4694-b893-b6769cf32056"
+					(reference "U1")
+					(unit 1)
+				)
+			)
+			(project "power"
+				(path "/ef47adc1-536f-4520-9ebd-fa1d01e89711/58fd429d-e8bc-4dae-9d70-752a4565c9e8/682a7ccb-ae4e-4e27-aa22-99379a5a65e4/fd3f1189-33c7-4694-b893-b6769cf32056"
+					(reference "U5")
 					(unit 1)
 				)
@@
 		(instances
 			(project "control"
-				(path "/c4b3c8f9-82bd-4648-8d22-870bf16aa829/29a81977-0a76-472b-8d88-45695e75b501/ace0dddc-e7de-4238-9577-ce744b7cdb3f/3f2d8199-33e9-456c-b5a1-16126a4e29ed"
-					(reference "C82")
-					(unit 1)
-				)
-				(path "/c4b3c8f9-82bd-4648-8d22-870bf16aa829/94383bfe-d869-4ac9-b660-9c199e344f31/9d3a0f9f-9dfc-4311-9915-9308a3fac81f/3f2d8199-33e9-456c-b5a1-16126a4e29ed"
+				(path "/c4b3c8f9-82bd-4648-8d22-870bf16aa829/29a81977-0a76-472b-8d88-45695e75b501/5d95f24e-69a0-4585-974a-64f0c2602c3c/fd3f1189-33c7-4694-b893-b6769cf32056"
+					(reference "C32")
+					(unit 1)
+				)
+				(path "/c4b3c8f9-82bd-4648-8d22-870bf16aa829/94383bfe-d869-4ac9-b660-9c199e344f31/9d3a0f9f-9dfc-4311-9915-9308a3fac81f/fd3f1189-33c7-4694-b893-b6769cf32056"
+					(reference "C30")
+					(unit 1)
+				)
+			)
+			(project "power"
+				(path "/ef47adc1-536f-4520-9ebd-fa1d01e89711/58fd429d-e8bc-4dae-9d70-752a4565c9e8/682a7ccb-ae4e-4e27-aa22-99379a5a65e4/fd3f1189-33c7-4694-b893-b6769cf32056"
 					(reference "C32")
 					(unit 1)
@@
 		(instances
 			(project "control"
-				(path "/c4b3c8f9-82bd-4648-8d22-870bf16aa829/29a81977-0a76-472b-8d88-45695e75b501/ace0dddc-e7de-4238-9577-ce744b7cdb3f/3f2d8199-33e9-456c-b5a1-16126a4e29ed"
-					(reference "C81")
-					(unit 1)
-				)
-				(path "/c4b3c8f9-82bd-4648-8d22-870bf16aa829/94383bfe-d869-4ac9-b660-9c199e344f31/9d3a0f9f-9dfc-4311-9915-9308a3fac81f/3f2d8199-33e9-456c-b5a1-16126a4e29ed"
+				(path "/c4b3c8f9-82bd-4648-8d22-870bf16aa829/29a81977-0a76-472b-8d88-45695e75b501/5d95f24e-69a0-4585-974a-64f0c2602c3c/fd3f1189-33c7-4694-b893-b6769cf32056"
 					(reference "C31")
 					(unit 1)
+				)
+				(path "/c4b3c8f9-82bd-4648-8d22-870bf16aa829/94383bfe-d869-4ac9-b660-9c199e344f31/9d3a0f9f-9dfc-4311-9915-9308a3fac81f/fd3f1189-33c7-4694-b893-b6769cf32056"
+					(reference "C1")
+					(unit 1)
+				)
+			)
+			(project "power"
+				(path "/ef47adc1-536f-4520-9ebd-fa1d01e89711/58fd429d-e8bc-4dae-9d70-752a4565c9e8/682a7ccb-ae4e-4e27-aa22-99379a5a65e4/fd3f1189-33c7-4694-b893-b6769cf32056"
+					(reference "C31")
+					(unit 1)
