File: COMMAND/KICAD/command.kicad_sch (KiCad schematic)
At the start: 0 parts

Commit message: Updated Command Kicad
Parts:
- added R4, R5: 4.7kΩ, Resistor_SMD:R_0603_1608Metric, symbol Device:R
Connections:
- new net I2C1.SCL: R4.2
- new net I2C1.SDA: R5.2
Other:
- added sheet EFUSE_LATCHED (../../POWER/KICAD/efuse.latched.kicad_sch)
- added sheet EXPANDER (expander.kicad_sch)
- sheet CAN ports: added CAN_I, CAN_O, STB, V_3.3; removed CAN, V_LV
- sheet DEBUG ports: added V_3.3; removed V_LV
- sheet MCU ports: added PB[0..15], PC[0..15], PD[0..15], PE[0..15], PH[0..3], RESET, V_3.3, V_BAT, {PA}; removed NRST, PA, PB
- note added: "BOOTLOADER"
- note added: "BOOTLOADER ON I2C1 / I2C2 / I2C3"
- note added: "CAN_STANDBY OPEN DRAIN"
- note added: "FDCAN TX: PD1 RX: PD0"
- note added: "FORCE CAN COMMUNICATION"
- note added: "FUSE"
- note added: "I2C1"
- note added: "I2C1 SCL: PB8 SDA: PB9"
- note added: "I2C2"
- note added: "I2C2 SCL: PB10 SDA: PB11"
- note added: "MASTER COMMUNICATION"
- note added: "RESET"
- note added: "SLAVE BACKUP COMMUNICATION"
- note added: "SWD SWCLK: PA14 SWDIO: PA13 SWO: PB3"
- note added: "USART RX: PA10 TX: PA9"
- note added: "USB DP: PA12 DM: PA11"

Commit message: schematic design
Parts:
- removed R4: 4.7kΩ, Resistor_SMD:R_0603_1608Metric, symbol Device:R
- added R18: 4.7kΩ, Resistor_SMD:R_0603_1608Metric, symbol Device:R
- added R38: R, symbol Device:R
Connections:
- net EFUSE_LATCHED/V_GND: now also R38.2
- net I2C1.SCL: now also R5.2
- net I2C1.SDA: now also R18.2; no longer R5.2
- new net EFUSE_LATCHED/I_LIM: R38.1
Other:
- added sheet SMPS(3.3 V) (../../POWER/KICAD/smps_3V3.kicad_sch)
- sheet DEBUG ports: added {SWD}, {UART}; removed DEBUG, UART
- sheet EFUSE_LATCHED ports: added ENABLE, I_LIM; removed none
- sheet MCU ports: added {PB}, {PC}, {PD}, {PE}, {PH}; removed PB[0..15], PC[0..15], PD[0..15], PE[0..15], PH[0..3]
- note added: "BACKUP/I2C"
- note added: "CAN"
- note added: "DEBUG"
- note added: "EXPANDER"
- note added: "POWER"
- note removed: "BOOTLOADER"
- note removed: "FUSE"
