File: COMMAND/KICAD/debug.kicad_sch (KiCad schematic)
At the start: 1 part

Commit message: Updated Command Kicad
Parts:
- gave numbers to parts that had none: 1
Connections:
- net V_LV renamed V_3.3
Changed lines of the file:
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@@
 		)
 	)
-	(hierarchical_label "UART"
+	(hierarchical_label "UART{TX RX}"
 		(shape input)
 		(at 199.39 113.03 0)
@@
 		)
 	)
-	(hierarchical_label "DEBUG"
+	(hierarchical_label "SWD{NRST SWDIO SWCLK SWO}"
 		(shape input)
 		(at 218.44 90.17 0)
@@
 		)
 	)
-	(hierarchical_label "V_LV"
+	(hierarchical_label "V_3.3"
 		(shape input)
 		(at 135.89 95.25 180)
@@
 		(on_board yes)
 		(dnp no)
-		(property "Reference" "J?"
+		(property "Reference" "J2"
 			(at 149.86 86.614 0)
 			(effects
@@
 		(instances
 			(project "control"
-				(path "/c4b3c8f9-82bd-4648-8d22-870bf16aa829/25a33f1f-9c89-41a2-a6e3-9fd3adab2d11/29e40f37-92ad-48d8-a826-f7dff8f4d82a"
-					(reference "J?")
+				(path "/c4b3c8f9-82bd-4648-8d22-870bf16aa829/29a81977-0a76-472b-8d88-45695e75b501/ace0dddc-e7de-4238-9577-ce744b7cdb3f/29e40f37-92ad-48d8-a826-f7dff8f4d82a"
+					(reference "J3")
 					(unit 1)
 				)
+				(path "/c4b3c8f9-82bd-4648-8d22-870bf16aa829/94383bfe-d869-4ac9-b660-9c199e344f31/9d3a0f9f-9dfc-4311-9915-9308a3fac81f/29e40f37-92ad-48d8-a826-f7dff8f4d82a"
+					(reference "J2")
+					(unit 1)
+				)

Commit message: schematic design
Parts:
- removed J2: FTSH-107-01-X-DV, symbol CUBESAT:FTSH-107-XX-X-DV
- added J3: Conn_02x07_Odd_Even, symbol Connector_Generic:Conn_02x07_Odd_Even
Connections:
- net V_3.3: now also J3.3 (Pin_3)
- net V_GND: now also J3.11 (Pin_11), J3.5 (Pin_5), J3.7 (Pin_7)
- new net NRST: J3.12 (Pin_12)
- new net RX: J3.13 (Pin_13)
- new net SWCLK: J3.6 (Pin_6)
- new net SWDIO: J3.4 (Pin_4)
- new net SWO: J3.8 (Pin_8)
- new net TX: J3.14 (Pin_14)
