File: COMMAND/KICAD/expander.kicad_sch (KiCad schematic)
At the start: 8 parts, among them U2 TCAL9538RSV

Commit message: schematic design
Parts:
- renumbered C2 to C?, R11 to R?, R9 to R?, R7 to R?, R10 to R?, R6 to R?, R8 to R?, U2 to U?
Connections:
- net I2C.SCL renamed SCL
- net I2C.SDA renamed SDA
