File: COMMAND/KICAD/temperature_sensor.kicad_sch (KiCad schematic)
At the start: 4 parts, among them U2 TMP112N

Commit message: schematic design
Parts:
- renumbered C2 to C10, R3 to R33, R4 to R34, U2 to U6
Changed lines of the file:
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@@
 		(dnp no)
 		(fields_autoplaced yes)
-		(property "Reference" "C2"
+		(property "Reference" "C10"
 			(at 110.49 99.0599 0)
 			(effects
@@
 		)
 		(instances
-			(project ""
-				(path "/d0cf13c6-7468-4a0f-ad0e-01e083e4d938/b8cd3b68-e49c-4009-8a50-5ec068f5cb3a"
-					(reference "C2")
-					(unit 1)
-				)
-			)
-			(project ""
-				(path "/ef47adc1-536f-4520-9ebd-fa1d01e89711/58fd429d-e8bc-4dae-9d70-752a4565c9e8/3638ca90-9701-4456-8013-6f74e8e57495"
-					(reference "C28")
+			(project "power"
+				(path "/ef47adc1-536f-4520-9ebd-fa1d01e89711/58fd429d-e8bc-4dae-9d70-752a4565c9e8/272627ea-7474-456d-81ae-5f6b1fdd0a68/2708a68d-1022-4340-b2e0-aa371803758b"
+					(reference "C10")
 					(unit 1)
 				)
@@
 		(dnp no)
 		(fields_autoplaced yes)
-		(property "Reference" "R4"
+		(property "Reference" "R34"
 			(at 179.07 101.5999 0)
 			(effects
@@
 		(instances
 			(project "power"
-				(path "/d0cf13c6-7468-4a0f-ad0e-01e083e4d938/b8cd3b68-e49c-4009-8a50-5ec068f5cb3a"
-					(reference "R4")
-					(unit 1)
-				)
-			)
-			(project "power"
-				(path "/ef47adc1-536f-4520-9ebd-fa1d01e89711/58fd429d-e8bc-4dae-9d70-752a4565c9e8/3638ca90-9701-4456-8013-6f74e8e57495"
+				(path "/ef47adc1-536f-4520-9ebd-fa1d01e89711/58fd429d-e8bc-4dae-9d70-752a4565c9e8/272627ea-7474-456d-81ae-5f6b1fdd0a68/2708a68d-1022-4340-b2e0-aa371803758b"
 					(reference "R34")
 					(unit 1)
@@
 		(dnp yes)
 		(fields_autoplaced yes)
-		(property "Reference" "R3"
+		(property "Reference" "R33"
 			(at 179.07 88.8999 0)
 			(effects
@@
 		(instances
 			(project "power"
-				(path "/d0cf13c6-7468-4a0f-ad0e-01e083e4d938/b8cd3b68-e49c-4009-8a50-5ec068f5cb3a"
-					(reference "R3")
-					(unit 1)
-				)
-			)
-			(project "power"
-				(path "/ef47adc1-536f-4520-9ebd-fa1d01e89711/58fd429d-e8bc-4dae-9d70-752a4565c9e8/3638ca90-9701-4456-8013-6f74e8e57495"
+				(path "/ef47adc1-536f-4520-9ebd-fa1d01e89711/58fd429d-e8bc-4dae-9d70-752a4565c9e8/272627ea-7474-456d-81ae-5f6b1fdd0a68/2708a68d-1022-4340-b2e0-aa371803758b"
 					(reference "R33")
 					(unit 1)
@@
 		(on_board yes)
 		(dnp no)
-		(property "Reference" "U2"
+		(property "Reference" "U6"
 			(at 153.67 88.9 0)
 			(effects
@@
 		)
 		(instances
-			(project ""
-				(path "/d0cf13c6-7468-4a0f-ad0e-01e083e4d938/b8cd3b68-e49c-4009-8a50-5ec068f5cb3a"
-					(reference "U2")
-					(unit 1)
-				)
-			)
-			(project ""
-				(path "/ef47adc1-536f-4520-9ebd-fa1d01e89711/58fd429d-e8bc-4dae-9d70-752a4565c9e8/3638ca90-9701-4456-8013-6f74e8e57495"
+			(project "power"
+				(path "/ef47adc1-536f-4520-9ebd-fa1d01e89711/58fd429d-e8bc-4dae-9d70-752a4565c9e8/272627ea-7474-456d-81ae-5f6b1fdd0a68/2708a68d-1022-4340-b2e0-aa371803758b"
 					(reference "U6")
 					(unit 1)
