File: COMMUNICATION/KICAD/attenuator.kicad_sch (KiCad schematic)
At the start: 1 part, among them U1 PAT1220-C-10DB

Commit message: schematic design
Parts:
- renumbered U1 to U9
Changed lines of the file:
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@@
 		(on_board yes)
 		(dnp no)
-		(property "Reference" "U1"
+		(property "Reference" "U9"
 			(at 151.13 83.566 0)
 			(effects
@@
 		(instances
 			(project "communication"
-				(path "/5d09a5b0-5470-41ee-acbf-63da99fdcb81/4eb0d389-8a08-4cbf-a5eb-8a7b63640ccd/831451b2-3007-47ac-a3e1-e45c9767ea10"
+				(path "/5d09a5b0-5470-41ee-acbf-63da99fdcb81/4eb0d389-8a08-4cbf-a5eb-8a7b63640ccd/a021a516-f8a2-48a4-8b79-b531761ea9b5"
 					(reference "U1")
 					(unit 1)
 				)
-				(path "/5d09a5b0-5470-41ee-acbf-63da99fdcb81/4eb0d389-8a08-4cbf-a5eb-8a7b63640ccd/c11b217c-e18a-4a41-8758-05d70ecb46e2"
-					(reference "U3")
+				(path "/5d09a5b0-5470-41ee-acbf-63da99fdcb81/4eb0d389-8a08-4cbf-a5eb-8a7b63640ccd/b90e1395-1e98-4e3a-bf33-85d3c9f53eb2"
+					(reference "U9")
 					(unit 1)
 				)
-				(path "/5d09a5b0-5470-41ee-acbf-63da99fdcb81/e60adf2b-68aa-469a-b511-2688a73729bb/831451b2-3007-47ac-a3e1-e45c9767ea10"
+				(path "/5d09a5b0-5470-41ee-acbf-63da99fdcb81/e60adf2b-68aa-469a-b511-2688a73729bb/a021a516-f8a2-48a4-8b79-b531761ea9b5"
 					(reference "U14")
 					(unit 1)
 				)
-				(path "/5d09a5b0-5470-41ee-acbf-63da99fdcb81/e60adf2b-68aa-469a-b511-2688a73729bb/c11b217c-e18a-4a41-8758-05d70ecb46e2"
+				(path "/5d09a5b0-5470-41ee-acbf-63da99fdcb81/e60adf2b-68aa-469a-b511-2688a73729bb/b90e1395-1e98-4e3a-bf33-85d3c9f53eb2"
 					(reference "U10")
 					(unit 1)
