File: COMMUNICATION/KICAD/communication.kicad_sch (KiCad schematic)
At the start: 4 parts

Commit message: schematic design
Parts:
- added J2: Conn_02x07_Odd_Even, symbol Connector_Generic:Conn_02x07_Odd_Even
- added J5: Conn_Coaxial, symbol Connector:Conn_Coaxial
Connections:
- net GND: now also J5.2 (Ext)
Other:
- moved on the sheet: H1, H2, H3, H4
