File: COMMUNICATION/KICAD/communication.module.kicad_sch (KiCad schematic)
At the start: 1 part

Commit message: schematic design
Connections:
- net MONITOR/OUT renamed V_5.0
- no-connect marks 1 -> 0
Other:
- added sheet EFUSE_LATCHED (../../POWER/KICAD/efuse.latched.kicad_sch)
- added sheet SMPS(5.0 V) (../../POWER/KICAD/smps_5V0.kicad_sch)
- sheet COMMAND ports: added V_IN, {CAN}, {I2C}, {PA}, {PB}, {PC}, {PD}, {PE}, {PH}; removed CAN, I2C, INT, PA, PB, PC, PD, PH
- sheet TRANSCIEVER ports: added DIO[1..2], ENABLE{RX TX}, {SPI}; removed DIO, ENABLE, SPI
- note added: "HV POWER"
- note added: "RF PATH"
- moved on the sheet: R13
