File: COMMUNICATION/KICAD/coupler.kicad_sch (KiCad schematic)
At the start: 1 part, among them U4 X4C09F1-30S

Commit message: schematic design
Parts:
- renumbered U4 to U3
Changed lines of the file:
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@@
 		(dnp no)
 		(fields_autoplaced yes)
-		(property "Reference" "U4"
+		(property "Reference" "U3"
 			(at 148.59 94.996 0)
 			(do_not_autoplace yes)
@@
 		(instances
 			(project "communication"
-				(path "/5d09a5b0-5470-41ee-acbf-63da99fdcb81/4eb0d389-8a08-4cbf-a5eb-8a7b63640ccd/d474d84d-c447-4bc2-aa61-4f57e1a8a903"
-					(reference "U4")
+				(path "/5d09a5b0-5470-41ee-acbf-63da99fdcb81/4eb0d389-8a08-4cbf-a5eb-8a7b63640ccd/503aa56d-040d-4678-bd81-08001f5a7e2d"
+					(reference "U3")
 					(unit 1)
 				)
-				(path "/5d09a5b0-5470-41ee-acbf-63da99fdcb81/e60adf2b-68aa-469a-b511-2688a73729bb/d474d84d-c447-4bc2-aa61-4f57e1a8a903"
-					(reference "U12")
+				(path "/5d09a5b0-5470-41ee-acbf-63da99fdcb81/e60adf2b-68aa-469a-b511-2688a73729bb/503aa56d-040d-4678-bd81-08001f5a7e2d"
+					(reference "U11")
 					(unit 1)
 				)
