File: COMMUNICATION/KICAD/detector.kicad_sch (KiCad schematic)
At the start: 3 parts, among them U6 LMV221

Commit message: schematic design
Parts:
- R3: value 100kΩ -> 135kΩ
- renumbered U6 to U4
Changed lines of the file:
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@@
 		(instances
 			(project "communication"
-				(path "/5d09a5b0-5470-41ee-acbf-63da99fdcb81/4eb0d389-8a08-4cbf-a5eb-8a7b63640ccd/5efc2ac6-6661-44e2-8b94-f2851e091db5"
+				(path "/5d09a5b0-5470-41ee-acbf-63da99fdcb81/4eb0d389-8a08-4cbf-a5eb-8a7b63640ccd/611ffc60-9e46-441d-ae7c-396a267ab426"
 					(reference "C1")
 					(unit 1)
 				)
-				(path "/5d09a5b0-5470-41ee-acbf-63da99fdcb81/4eb0d389-8a08-4cbf-a5eb-8a7b63640ccd/7f6487ca-8c06-43f6-ab32-f7086d3a45c4"
-					(reference "C19")
+				(path "/5d09a5b0-5470-41ee-acbf-63da99fdcb81/4eb0d389-8a08-4cbf-a5eb-8a7b63640ccd/b38a137a-6f64-4fbf-b6b0-3363b61c2955"
+					(reference "C2")
 					(unit 1)
 				)
-				(path "/5d09a5b0-5470-41ee-acbf-63da99fdcb81/e60adf2b-68aa-469a-b511-2688a73729bb/5efc2ac6-6661-44e2-8b94-f2851e091db5"
-					(reference "C22")
+				(path "/5d09a5b0-5470-41ee-acbf-63da99fdcb81/e60adf2b-68aa-469a-b511-2688a73729bb/611ffc60-9e46-441d-ae7c-396a267ab426"
+					(reference "C3")
 					(unit 1)
 				)
-				(path "/5d09a5b0-5470-41ee-acbf-63da99fdcb81/e60adf2b-68aa-469a-b511-2688a73729bb/7f6487ca-8c06-43f6-ab32-f7086d3a45c4"
-					(reference "C21")
+				(path "/5d09a5b0-5470-41ee-acbf-63da99fdcb81/e60adf2b-68aa-469a-b511-2688a73729bb/b38a137a-6f64-4fbf-b6b0-3363b61c2955"
+					(reference "C4")
 					(unit 1)
 				)
@@
 			)
 		)
-		(property "Value" "100kΩ"
+		(property "Value" "135kΩ"
 			(at 181.61 104.1399 0)
 			(effects
@@
 		(instances
 			(project "communication"
-				(path "/5d09a5b0-5470-41ee-acbf-63da99fdcb81/4eb0d389-8a08-4cbf-a5eb-8a7b63640ccd/5efc2ac6-6661-44e2-8b94-f2851e091db5"
+				(path "/5d09a5b0-5470-41ee-acbf-63da99fdcb81/4eb0d389-8a08-4cbf-a5eb-8a7b63640ccd/611ffc60-9e46-441d-ae7c-396a267ab426"
 					(reference "R3")
 					(unit 1)
 				)
-				(path "/5d09a5b0-5470-41ee-acbf-63da99fdcb81/4eb0d389-8a08-4cbf-a5eb-8a7b63640ccd/7f6487ca-8c06-43f6-ab32-f7086d3a45c4"
+				(path "/5d09a5b0-5470-41ee-acbf-63da99fdcb81/4eb0d389-8a08-4cbf-a5eb-8a7b63640ccd/b38a137a-6f64-4fbf-b6b0-3363b61c2955"
 					(reference "R4")
 					(unit 1)
 				)
-				(path "/5d09a5b0-5470-41ee-acbf-63da99fdcb81/e60adf2b-68aa-469a-b511-2688a73729bb/5efc2ac6-6661-44e2-8b94-f2851e091db5"
-					(reference "R19")
+				(path "/5d09a5b0-5470-41ee-acbf-63da99fdcb81/e60adf2b-68aa-469a-b511-2688a73729bb/611ffc60-9e46-441d-ae7c-396a267ab426"
+					(reference "R10")
 					(unit 1)
 				)
-				(path "/5d09a5b0-5470-41ee-acbf-63da99fdcb81/e60adf2b-68aa-469a-b511-2688a73729bb/7f6487ca-8c06-43f6-ab32-f7086d3a45c4"
-					(reference "R18")
+				(path "/5d09a5b0-5470-41ee-acbf-63da99fdcb81/e60adf2b-68aa-469a-b511-2688a73729bb/b38a137a-6f64-4fbf-b6b0-3363b61c2955"
+					(reference "R11")
 					(unit 1)
 				)
@@
 		(dnp no)
 		(fields_autoplaced yes)
-		(property "Reference" "U6"
+		(property "Reference" "U4"
 			(at 143.51 91.186 0)
 			(do_not_autoplace yes)
@@
 		(instances
 			(project "communication"
-				(path "/5d09a5b0-5470-41ee-acbf-63da99fdcb81/4eb0d389-8a08-4cbf-a5eb-8a7b63640ccd/5efc2ac6-6661-44e2-8b94-f2851e091db5"
-					(reference "U6")
+				(path "/5d09a5b0-5470-41ee-acbf-63da99fdcb81/4eb0d389-8a08-4cbf-a5eb-8a7b63640ccd/611ffc60-9e46-441d-ae7c-396a267ab426"
+					(reference "U4")
 					(unit 1)
 				)
-				(path "/5d09a5b0-5470-41ee-acbf-63da99fdcb81/4eb0d389-8a08-4cbf-a5eb-8a7b63640ccd/7f6487ca-8c06-43f6-ab32-f7086d3a45c4"
+				(path "/5d09a5b0-5470-41ee-acbf-63da99fdcb81/4eb0d389-8a08-4cbf-a5eb-8a7b63640ccd/b38a137a-6f64-4fbf-b6b0-3363b61c2955"
 					(reference "U8")
 					(unit 1)
 				)
-				(path "/5d09a5b0-5470-41ee-acbf-63da99fdcb81/e60adf2b-68aa-469a-b511-2688a73729bb/5efc2ac6-6661-44e2-8b94-f2851e091db5"
-					(reference "U15")
+				(path "/5d09a5b0-5470-41ee-acbf-63da99fdcb81/e60adf2b-68aa-469a-b511-2688a73729bb/611ffc60-9e46-441d-ae7c-396a267ab426"
+					(reference "U12")
 					(unit 1)
 				)
-				(path "/5d09a5b0-5470-41ee-acbf-63da99fdcb81/e60adf2b-68aa-469a-b511-2688a73729bb/7f6487ca-8c06-43f6-ab32-f7086d3a45c4"
+				(path "/5d09a5b0-5470-41ee-acbf-63da99fdcb81/e60adf2b-68aa-469a-b511-2688a73729bb/b38a137a-6f64-4fbf-b6b0-3363b61c2955"
 					(reference "U13")
 					(unit 1)
