File: COMMUNICATION/KICAD/transciever.kicad_sch (KiCad schematic)
At the start: 1 part, among them U11 E22-400M30S

Commit message: schematic design
Parts:
- renumbered U11 to U6
Connections:
- net SPI.CS renamed CS
- net SPI.SCLK renamed SCK
- net SPI.SDI renamed SDI
- net SPI.SDO renamed SDO
Changed lines of the file:
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@@
 	(generator_version "8.0")
 	(paper "A4")
+	(bus_alias "SPI"
+		(members "SCK" "SDI" "SDO" "CS")
+	)
 	(junction
 		(at 143.51 102.87)
@@
 	(bus
 		(pts
-			(xy 71.12 86.36) (xy 97.79 86.36)
+			(xy 87.63 86.36) (xy 97.79 86.36)
 		)
 		(stroke
@@
 		)
 	)
-	(label "SPI{CS SCLK SDI SDO}"
+	(label "{SPI}"
 		(at 95.25 86.36 180)
 		(fields_autoplaced yes)
@@
 		)
 	)
-	(label "SPI.SDI"
+	(label "SDI"
 		(at 113.03 95.25 180)
 		(fields_autoplaced yes)
@@
 		)
 	)
-	(label "SPI.CS"
+	(label "CS"
 		(at 113.03 90.17 180)
 		(fields_autoplaced yes)
@@
 		)
 	)
-	(label "SPI.SDO"
+	(label "SDO"
 		(at 113.03 97.79 180)
 		(fields_autoplaced yes)
@@
 		)
 	)
-	(label "SPI.SCLK"
+	(label "SCK"
 		(at 113.03 92.71 180)
 		(fields_autoplaced yes)
@@
 		)
 	)
-	(hierarchical_label "ENABLE"
+	(hierarchical_label "ENABLE{RX TX}"
 		(shape input)
 		(at 78.74 99.06 180)
@@
 		)
 	)
-	(hierarchical_label "DIO"
+	(hierarchical_label "DIO[1..2]"
 		(shape bidirectional)
 		(at 167.64 85.09 0)
@@
 		)
 	)
-	(hierarchical_label "SPI{CS SCLK SDI SDO}"
+	(hierarchical_label "{SPI}"
 		(shape bidirectional)
-		(at 71.12 86.36 180)
+		(at 87.63 86.36 180)
 		(fields_autoplaced yes)
 		(effects
@@
 		(on_board yes)
 		(dnp no)
-		(property "Reference" "U11"
+		(property "Reference" "U6"
 			(at 128.27 77.216 0)
 			(do_not_autoplace yes)
@@
 		(instances
 			(project "communication"
-				(path "/5d09a5b0-5470-41ee-acbf-63da99fdcb81/4eb0d389-8a08-4cbf-a5eb-8a7b63640ccd/db0bc37c-7e2e-4192-a9ef-5d3860346c8a"
-					(reference "U11")
+				(path "/5d09a5b0-5470-41ee-acbf-63da99fdcb81/4eb0d389-8a08-4cbf-a5eb-8a7b63640ccd/0e426de6-47a4-4e57-a06e-750b655f3261"
+					(reference "U6")
 					(unit 1)
 				)
-				(path "/5d09a5b0-5470-41ee-acbf-63da99fdcb81/e60adf2b-68aa-469a-b511-2688a73729bb/db0bc37c-7e2e-4192-a9ef-5d3860346c8a"
-					(reference "U16")
+				(path "/5d09a5b0-5470-41ee-acbf-63da99fdcb81/e60adf2b-68aa-469a-b511-2688a73729bb/0e426de6-47a4-4e57-a06e-750b655f3261"
+					(reference "U15")
 					(unit 1)
 				)
