File: POWER/KICAD/battery.module.kicad_sch (KiCad schematic)
At the start: 9 parts, among them U10 ISO1541, U7 BQ76905

Commit message: schematic design
Other:
- note added: "HEATER"
- note added: "PROTECTOR / BALANCER / MONITOR"
- note added: "TEMP SENSOR"
- note added: "TEST POINTS FOR BATTERY ALONG JUMPERS TO HANDLE BATTERIES TEST POINTS TO CHARGE BATTERIES EXTERNALLY?"
- note added: "TEST POINTS TO SIMULATE BATTERY"
Changed lines of the file:
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@@
+		)
+	)
+	(rectangle
+		(start -7.62 149.86)
+		(end 177.8 236.22)
+		(stroke
+			(width 0)
+			(type default)
+		)
+		(fill
+			(type none)
+		)
+	)
+	(rectangle
+		(start 106.68 50.8)
+		(end 292.1 137.16)
+		(stroke
+			(width 0)
+			(type default)
+		)
+		(fill
+			(type none)
+		)
+	)
+	(text "TEMP SENSOR"
+		(exclude_from_sim no)
+		(at 2.54 160.02 0)
+		(effects
+			(font
+				(size 1.27 1.27)
+			)
+			(justify left top)
+		)
+	)
+	(text "PROTECTOR / BALANCER / MONITOR"
+		(exclude_from_sim no)
+		(at 109.22 53.34 0)
+		(effects
+			(font
+				(size 1.27 1.27)
+			)
+			(justify left top)
+		)
+	)
+	(text "TEST POINTS TO SIMULATE BATTERY"
+		(exclude_from_sim no)
+		(at 170.18 71.12 0)
+		(effects
+			(font
+				(size 1.27 1.27)
+			)
+			(justify left top)
+		)
+	)
+	(text "HEATER"
+		(exclude_from_sim no)
+		(at -5.08 152.4 0)
+		(effects
+			(font
+				(size 1.27 1.27)
+			)
+			(justify left top)
+		)
+	)
+	(text "TEST POINTS FOR BATTERY ALONG JUMPERS TO HANDLE BATTERIES\nTEST POINTS TO CHARGE BATTERIES EXTERNALLY?"
+		(exclude_from_sim no)
+		(at 170.18 63.5 0)
+		(effects
+			(font
+				(size 1.27 1.27)
+			)
+			(justify left top)
 		)
 	)
