File: POWER/KICAD/efuse.retry.kicad_sch (KiCad schematic)
At the start: 6 parts, among them U2 TPS24701 RETRY

Commit message: schematic design
Parts:
- removed C3, C6: 100nF, symbol Device:C
- removed C4: 68nF, symbol Device:C
- removed D2: D_Zener, symbol Device:D_Zener
- removed R1: 4.7kΩ, symbol Device:R
- removed U2: TPS24701 RETRY, symbol CUBESAT:TPS24701
- added R46: 30kΩ, symbol Device:R
- added R47, R52: 4.7kΩ, symbol Device:R
- added U?: TPS259474A, symbol CUBESAT:TPS259474ARPW
Connections:
- net EN: now also R46.2, R47.1, U?.1 (EN/UVLO)
- net V_GND: now also R52.2
- net V_IN: now also R46.1, U?.5 (IN)
- net V_OUT: now also U?.6 (OUT)
- new net PG: U?.3 (PG)
- new net UVLO: R47.2, R52.1, U?.2 (OVLO)
Other:
- removed sheet QFET
- note added: "CURRENT LIMIT R = 3334 / I"
- note added: "OV: 11 V UV: 5.6 V"
- note removed: "C_TIMER = (10uA) / (1.35V) * T_FLT"
- note removed: "C_TIMER = 68 nF"
- note removed: "INPUT CAPACITOR"
- note removed: "OUTPUT CAPACITOR"
- note removed: "PULL-UP RESISTOR"
- note removed: "QFET FOR RELIABILITY / REDUNDANCY"
- note removed: "T_FLT = 9.8 ms"
- note removed: "T_FLT = ~ 10 ms"
- note removed: "ZENER CLAMPS VOLTAGE"
