File: POWER/KICAD/mppt.kicad_sch (KiCad schematic)
At the start: 13 parts, among them U3 TPS61376

Commit message: schematic design
Parts:
- removed C9: ~, symbol Device:C
- added C3, C4: 22uF, symbol Device:C
- added D2, D7: D_Schottky, symbol Device:D_Schottky
- added Q2: 2N7002, Package_TO_SOT_SMD:SOT-23, symbol Transistor_FET:2N7002
- added R28: 220 kΩ, symbol Device:R
- added R30, R38: 135 kΩ, symbol Device:R
- added R32, R35: 0 kΩ, symbol Device:R
- added R40, R42, R43: 4.7kΩ, Resistor_SMD:R_0603_1608Metric, symbol Device:R
- R10, R13: value R -> 30 kΩ
- R11: value R -> 4.7kΩ; footprint (none) -> Resistor_SMD:R_0603_1608Metric
- R12: value R -> 220 kΩ
Connections:
- net SHUTDOWN: now also D7.1 (K)
- net V_GND: now also C3.2, C4.2, Q2.2 (S), R28.2, R30.2, R38.2, R40.2, R43.2; no longer R11.1
- net V_IN: now also L1.1, R42.1; no longer L1.2
- net V_OUT: now also C3.1, C4.1
- net at U3.5 (VP): now also L1.2; no longer L1.1
- net ILIM: now reaches U3.10 (ILIM)
- net ILIM: now also D2.1 (K), Q2.3 (D), R28.1, R30.1, R32.2
- net EN: now reaches R10.2, U3.2 (EN/UVLO)
- net EN: now also R11.1, D7.2 (A); no longer R11.2
- net ISEL: now reaches U3.3 (ISEL)
- net ISEL: now also R42.2, R43.1
- net COMP: now reaches U3.9 (COMP)
- new net: R11.2, R40.1
- new net: D2.2 (A), R32.1, R35.2
- new net CURRENT: Q2.1 (G), R35.1, R38.1
Other:
- note added: "135 + 220 = 83"
- note added: "CAPACITORS"
- note added: "COMP"
- note added: "COMPENSATION LOOP"
- note added: "CURRENT LIMIT"
- note added: "CURRENT LIMIT(ILIM): HIGH(ISEL > 0.84 V) 43.2 KΩ / 0.1 = 432 KΩ 43.2 KΩ / 3.0 = 14.4 KΩ LOW(ISEL < 0.84) 10.8 KΩ / 0.1 = 108 KΩ 10.8 KΩ / 0.75 = 14.4 KΩ UNSUPERVISED I = 0.5 A = 43.2 KΩ / 0.45 A = 81 KΩ ~= 130 + 220 KΩ = 0.51 A SUPERVISED = I = 0.9 A = 43.2 KΩ / 0.9 A = 48 KΩ ~= 120 KΩ"
- note added: "CURRENT VCC: 10 mA PEAK: 4.5 A (ISEL = HIGH) (1.005 A) CONTINOUS: 3 A (0.945 A) (0.5 A Unsupervised) LIMIT: 0.1 A ~ 3A"
- note added: "ENABLE W SHUTDOWN"
- note added: "INPUT"
- note added: "ISEL"
- note added: "OUTPUT"
- note added: "R1 = ((V_OUT - V_REF) * R2) / V_REF V_OUT = 8.4 V_REF = 1 R2 = 30 KΩ < 500 KΩ R1 = (7.4) * 30 KΩ = 222 KΩ ~= 220 KΩ"
- note added: "SUPERVISED"
- note added: "SUPERVISED(BACKUP)"
- note added: "UNSUPERVISED"
- note added: "USING MOSFET IN OHMIC REGION OR PWM IF THIS DOESN'T WORK OR IS IN ACCURATE USE THE SECOND OPTION BY SOLDERING RESISTOR THEN REMOVE DIODE IF ILIM NEVER EXCEEDS STM32 DAC I WILL SACRIFICE A BOARD ONCE ILIM IS TESTED"
- note added: "VOLTAGE IN: 2.9 V ~ 23 V (3 V ~ 6 V) VCC: 4.8 V VREF: (1V) ENABLE: >0.835 V"
- note added: "V_IN_ON = 0.813 * (1+R1/R2) V_IN_ON = 3.4V R1 = 30K R2 = 4.7 * 2 K DELTA = R1 * I_UVLO I_UVLO = 2 * 10^-6 mA DELTA = 0.06 V"
- note removed: "CURRENT VCC: 10 mA PEAK: 4.5 A CONTINOUS: 3 A LIMIT: 0.1 A ~ 3A"
- note removed: "ILIM: HIGH: 43.2 KΩ / 0.1 = 432 KΩ 43.2 KΩ / 3.0 = 14.4 KΩ LOW: 10.8 KΩ / 0.1 = 108 KΩ 10.8 KΩ / 0.75 = 14.4 KΩ"
- note removed: "ISEL = HIGH 4.5 A peak"
- note removed: "R1 = ((V_OUT - V_REF) * R2) / V_REF"
- note removed: "SHORT V_IN = 6 6 * 1.05 + 0.2 = 6.5"
- note removed: "VOLTAGE VCC: 4.8 V VREF: 1V ENABLE: 0.835 V"
- note removed: "V_IN_ON = 0.813 * (1+R1/R2) V_IN_ON = 4? 3? R1 = 10K R2 = 4.7K DELTA = R1 * I_UVLO I_UVLO = 2 * 10^-6 mA"
- moved on the sheet: C7, C8, D1, L1, R12, R13, U3
